File: MB1180/MCU_32-SchDoc.kicad_sch (KiCad schematic)
At the start: 52 parts, among them CN3 Header 15X1_male, CN4 Header 15X1_male, U2 MCU_LQFP32/QFN32, U3 LD39050PU33R, U5V_ST_LINK U5V_ST_LINK, U6 LD1117S50TR, X1 NX3215SA-32.768K-EXS00A-MU005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

Commit message: add some components
Parts:
- SB10, SB11, SB12, SB13, SB14, SB15, SB16, SB17, SB18, SB4, SB5, SB6, SB7, SB8: value (none) -> ~
Changed lines of the file:
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@@
       (effects (font (size 1.524 1.524)) (justify left bottom))
     )
-    (property "Value" "" (at 45.72 69.85 0)
+    (property "Value" "~" (at 45.72 69.85 0)
       (effects (font (size 1.27 1.27)) hide)
     )
@@
       (effects (font (size 1.524 1.524)) (justify left bottom))
     )
-    (property "Value" "" (at 254 123.19 0)
+    (property "Value" "~" (at 254 123.19 0)
       (effects (font (size 1.27 1.27)) hide)
     )
@@
       (effects (font (size 1.524 1.524)) (justify left bottom))
     )
-    (property "Value" "" (at 254 120.65 0)
+    (property "Value" "~" (at 254 120.65 0)
       (effects (font (size 1.27 1.27)) hide)
     )
@@
       (effects (font (size 1.524 1.524)) (justify left bottom))
     )
-    (property "Value" "" (at 48.26 6.35 0)
+    (property "Value" "~" (at 48.26 6.35 0)
       (effects (font (size 1.27 1.27)) hide)
     )
@@
       (effects (font (size 1.524 1.524)) (justify left bottom))
     )
-    (property "Value" "" (at 45.72 54.61 0)
+    (property "Value" "~" (at 45.72 54.61 0)
       (effects (font (size 1.27 1.27)) hide)
     )
@@
       (effects (font (size 1.524 1.524)) (justify left bottom))
     )
-    (property "Value" "" (at 116.84 158.75 0)
+    (property "Value" "~" (at 116.84 158.75 0)
       (effects (font (size 1.27 1.27)) hide)
     )
@@
       (effects (font (size 1.524 1.524)) (justify right top))
     )
-    (property "Value" "" (at 241.3 156.21 0)
+    (property "Value" "~" (at 241.3 156.21 0)
       (effects (font (size 1.27 1.27)) hide)
     )
@@
       (effects (font (size 1.524 1.524)) (justify left bottom))
     )
-    (property "Value" "" (at 139.7 59.69 0)
+    (property "Value" "~" (at 139.7 59.69 0)
       (effects (font (size 1.27 1.27)) hide)
     )
@@
       (effects (font (size 1.524 1.524)) (justify left bottom))
     )
-    (property "Value" "" (at 157.48 16.51 0)
+    (property "Value" "~" (at 157.48 16.51 0)
       (effects (font (size 1.27 1.27)) hide)
     )
@@
       (effects (font (size 1.524 1.524)) (justify left bottom))
     )
-    (property "Value" "" (at 45.72 64.77 0)
+    (property "Value" "~" (at 45.72 64.77 0)
       (effects (font (size 1.27 1.27)) hide)
     )
@@
       (effects (font (size 1.524 1.524)) (justify left bottom))
     )
-    (property "Value" "" (at 160.02 46.99 0)
+    (property "Value" "~" (at 160.02 46.99 0)
       (effects (font (size 1.27 1.27)) hide)
     )
@@
       (effects (font (size 1.524 1.524)) (justify left bottom))
     )
-    (property "Value" "" (at 48.26 95.25 0)
+    (property "Value" "~" (at 48.26 95.25 0)
       (effects (font (size 1.27 1.27)) hide)
     )
@@
       (effects (font (size 1.524 1.524)) (justify left bottom))
     )
-    (property "Value" "" (at 157.48 31.75 0)
+    (property "Value" "~" (at 157.48 31.75 0)
       (effects (font (size 1.27 1.27)) hide)
     )
@@
       (effects (font (size 1.524 1.524)) (justify left bottom))
     )
-    (property "Value" "" (at 48.26 85.09 0)
-      (effects (font (size 1.27 1.27)) hide)
-    )
+    (property "Value" "~" (at 48.26 85.09 0)
+      (effects (font (size 1.27 1.27)) hide)
+    )
