File: MB1180/ST_LINK_V2-1-SCHDOC.kicad_sch (KiCad schematic)
At the start: 66 parts, among them CN1 1050170001, CN2 [N/A], T1 9013, U1 ST890CDR, U4 LD3985M33R, U5 STM32F103CBT6, U5V U5V, U5V_2 U5V, U5V_3 U5V, U5V_4 U5V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

Commit message: Link Nucleo32 into main HW project
Connections:
- net at R17.1: now also LD1.4
- net at R19.2: now also LD1.3
- net at R18.2: now also LD1.2
- net at R4.2: no longer R3.1
- net at R3.2: now also R4.1, T1.2 (B)
- net at R11.1: no longer R10.2
- new net: R10.1, R11.2, SB1.2
- new net: R3.1, R4.2
- new net: R10.2, R11.1
- now unconnected: R10.1, R11.2, R4.1

Commit message: add some components
Parts:
- SB1, SB2, SB3, SB9: value (none) -> ~
Connections:
- net at R17.1: now also LD1.4
- net at R19.2: now also LD1.3
- net at R18.2: now also LD1.2
- net at R4.2: no longer R3.1
- net at R3.2: now also R4.1, T1.2 (B)
- net at R11.1: no longer R10.2
- new net: R10.1, R11.2, SB1.2
- new net: R3.1, R4.2
- new net: R10.2, R11.1
- now unconnected: R10.1, R11.2, R4.1
Changed lines of the file:
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@@
       (effects (font (size 1.524 1.524)) (justify left bottom))
     )
-    (property "Value" "" (at 219.71 19.05 0)
+    (property "Value" "~" (at 219.71 19.05 0)
       (effects (font (size 1.27 1.27)) hide)
     )
@@
       (effects (font (size 1.524 1.524)) (justify left bottom))
     )
-    (property "Value" "" (at 90.17 19.05 0)
+    (property "Value" "~" (at 90.17 19.05 0)
       (effects (font (size 1.27 1.27)) hide)
     )
@@
       (effects (font (size 1.524 1.524)) (justify left bottom))
     )
-    (property "Value" "" (at 41.91 115.57 0)
+    (property "Value" "~" (at 41.91 115.57 0)
       (effects (font (size 1.27 1.27)) hide)
     )
@@
       (effects (font (size 1.524 1.524)) (justify left bottom))
     )
-    (property "Value" "" (at 41.91 105.41 0)
+    (property "Value" "~" (at 41.91 105.41 0)
       (effects (font (size 1.27 1.27)) hide)
     )
